File: PCB/weerstasie.kicad_pcb (KiCad board)
At the start: 2 copper layers, 10 parts, among them J1 RJ12, J2 batt -, J3 batt +, J4 RJ12, U1 BME280, U2 RFM95

Commit message: Add missing connections in schematic
Parts:
- added 10k1: R, Resistors_SMD:R_0805, F.Cu at (178.3, 51.6)
- added 10k2: R, Resistors_SMD:R_0805, F.Cu at (191.3, 57.3)
- added 10k3: R, Resistors_SMD:R_0805, F.Cu at (163.8, 50.4)
- added C10: 100nF, Capacitors_SMD:C_0805, F.Cu at (99.1, 146.4)
- added C11: 100nF, Capacitors_SMD:C_0805, F.Cu at (116.6, 147.2)
- added C12: 100nF, Capacitors_SMD:C_0805, F.Cu at (77.7, 101.1)
- added C2: 22p, Capacitors_SMD:C_0805, F.Cu at (188.2, 77.1)
- added C3: 22p, Capacitors_SMD:C_0805, F.Cu at (76.6, 114.4)
- added C4: 22p, Capacitors_SMD:C_0805, F.Cu at (166.9, 123.2)
- added C5: C_Small, Capacitors_SMD:C_0805, F.Cu at (151.3, 39.0)
- added C6: C_Small, Capacitors_SMD:C_0805, F.Cu at (76.6, 128.9)
- added C7: C_Small, Capacitors_SMD:C_0805, F.Cu at (83.8, 141.5)
- added C8: 100nF, Capacitors_SMD:C_0805, F.Cu at (151.6, 83.9)
- added C9: 100nF, Capacitors_SMD:C_0805, F.Cu at (85.3, 82.4)
- added J5: ICSP, Pin_Headers:Pin_Header_Straight_2x03_Pitch2.54mm, F.Cu at (102.1, 70.1)
- added J6: Battery, Pin_Headers:Pin_Header_Straight_1x02_Pitch2.54mm, F.Cu at (75.4, 88.1)
- added R1: 10k, Resistors_SMD:R_0805, F.Cu at (81.5, 47.4)
- added SW1: SW_Push, Buttons_Switches_SMD:SW_SPST_B3SL-1002P, F.Cu at (103.9, 63.6)
- added U3: ATMEGA1284P-AU, Housings_QFP:TQFP-44_10x10mm_Pitch0.8mm, F.Cu at (171.8, 83.2)
- added Y1: 8MHz, Crystals:Crystal_HC49-U_Vertical, F.Cu at (161.9, 104.5)
- J1: value RJ12 -> WIND
- J4: value RJ12 -> RAIN
Connections:
- J1 pad 2: (no net) -> /WIND_DIR
- J1 pad 3: (no net) -> /WIND_SPEED
- J1 pad 4: (no net) -> GND
- J1 pad 5: (no net) -> GND
- J2 pad 1: (no net) -> GND
- J3 pad 1: (no net) -> VCC
- J4 pad 3: (no net) -> /RAIN
- J4 pad 4: (no net) -> GND
- U1 pad 1: Net-(U1-Pad1) -> GND
- U1 pad 2: Net-(U1-Pad2) -> /BME_SS
- U1 pad 3: Net-(U1-Pad3) -> /MOSI
- U1 pad 4: Net-(U1-Pad4) -> /SCK
- U1 pad 5: Net-(U1-Pad5) -> /MISO
- U1 pad 6: Net-(U1-Pad6) -> VCC
- U1 pad 7: Net-(U1-Pad7) -> GND
- U1 pad 8: Net-(U1-Pad8) -> VCC
- U2 pad 1: (no net) -> GND
- U2 pad 10: (no net) -> GND
- U2 pad 13: (no net) -> VCC
- U2 pad 14: (no net) -> /RFM_D0
- U2 pad 15: (no net) -> /RFM_D1
- U2 pad 16: (no net) -> /RFM_D2
- U2 pad 2: (no net) -> /MISO
- U2 pad 3: (no net) -> /MOSI
- U2 pad 4: (no net) -> /SCK
- U2 pad 5: (no net) -> /RFM_SS
- U2 pad 6: (no net) -> /RFM_RESET
- U2 pad 8: (no net) -> GND
Routing:
- net Net-(C1-Pad1): track 7.62 -> 20.6 mm, vias 0 -> 1
- net VCC: track 0.00 -> 2.67 mm
- net GND: track 0.00 -> 2.67 mm
- net Net-(U1-Pad8): track 1.41 -> 0.00 mm
- net Net-(U1-Pad1): track 1.41 -> 0.00 mm
- net Net-(U1-Pad5): track 1.36 -> 0.00 mm
- net Net-(U1-Pad4): track 1.36 -> 0.00 mm
- net /SCK: track 0.00 -> 1.36 mm
- net /MISO: track 0.00 -> 1.36 mm
- net Net-(U1-Pad7): track 1.26 -> 0.00 mm
- net Net-(U1-Pad6): track 1.26 -> 0.00 mm
- net Net-(U1-Pad3): track 1.16 -> 0.00 mm
- net Net-(U1-Pad2): track 1.16 -> 0.00 mm
- net /MOSI: track 0.00 -> 1.16 mm
- net /BME_SS: track 0.00 -> 1.16 mm

Commit message: Ready to be routed
Parts:
- removed 10k2, 10k3: R, Resistors_SMD:R_0805
- removed the J6 at (75.4, 88.1)
- removed the R1 at (81.5, 47.4)
- added C4: 100n, Capacitors_SMD:C_0805, F.Cu at (126.5, 64.1)
- added J5: SolarSensJumpers, Pin_Headers:Pin_Header_Straight_2x04_Pitch1.00mm, F.Cu at (126.6, 114.9)
- added J7: INT2, Pin_Headers:Pin_Header_Straight_1x01_Pitch2.54mm, F.Cu at (191.4, 103.6)
- added J8: I2C, Pin_Headers:Pin_Header_Straight_1x02_Pitch2.54mm, F.Cu at (191.5, 116.3)
- added J9: UART, Pin_Headers:Pin_Header_Straight_1x02_Pitch2.54mm, F.Cu at (191.4, 108.2)
- added R2: 10k2, Resistors_SMD:R_0805, F.Cu at (155.1, 40.0)
- added R3: 10k3, Resistors_SMD:R_0805, F.Cu at (157.1, 40.0)
- added R4: 10k, Resistors_SMD:R_0805, F.Cu at (159.4, 75.6)
- C1: renamed from C2; value 22p -> 100n
- C2: renamed from C3; value 22p -> 100n
- C3: renamed from C4; value 22p -> 100n
- C5: value C_Small -> 100n
- C7: renamed from C6; value C_Small -> 22p
- C8: renamed from C7; value C_Small -> 22p
- J2, J3: footprint Pin_Headers:Pin_Header_Straight_1x01_Pitch2.54mm -> drawn_by_jpmeijers:BATTERY_TERMINAL
- R1: renamed from 10k1; value R -> 10k1
- moved C2 105.9 mm to (155.1, 43.3), turned to 270 degrees
- moved C13 104.1 mm to (180.3, 83.7)
- moved C7 92.4 mm to (166.9, 109.2), turned to 270 degrees
- moved C11 91.3 mm to (172.1, 91.7), turned to 270 degrees
- moved C10 87.3 mm to (172.3, 74.7), turned to 90 degrees
- moved C8 84.5 mm to (161.9, 109.2), turned to 270 degrees
- moved C3 80.5 mm to (157.1, 43.3), turned to 270 degrees
- moved C12 79.7 mm to (163.3, 82.7), turned to 180 degrees
- moved C5 62.6 mm to (112.8, 88.4), turned to 90 degrees
- moved SW1 51.7 mm to (154.8, 72.6)
- moved C1 48.8 mm to (153.0, 43.3), turned to 270 degrees
- moved C9 28.8 mm to (180.3, 82.0)
- moved R1 27.8 mm to (153.0, 40.0), turned to 270 degrees
- moved J2 4.92 mm to (109.5, 131.0)
- moved J3 4.03 mm to (125.5, 131.0)
- renumbered C9 to C10, C10 to C11, C11 to C12, C12 to C13, C1 to C6, C8 to C9, J5 to J6
Connections:
- J4 pad 1: (no net) -> Net-(J4-Pad1)
- J4 pad 2: (no net) -> Net-(J4-Pad2)
- J4 pad 5: (no net) -> Net-(J4-Pad5)
- J4 pad 6: (no net) -> Net-(J4-Pad6)
- U3 pad 10: (no net) -> Net-(J9-Pad2)
- U3 pad 19: /RFM_D0 -> Net-(J8-Pad1)
- U3 pad 20: /RFM_D1 -> Net-(J8-Pad2)
- U3 pad 21: /RFM_D2 -> /RFM_D0
- U3 pad 22: (no net) -> /RFM_D1
- U3 pad 23: (no net) -> /RFM_D2
- U3 pad 24: (no net) -> /RFM_RESET
- U3 pad 30: (no net) -> /SOLAR_6
- U3 pad 31: (no net) -> /SOLAR_5
- U3 pad 32: (no net) -> /SOLAR_2
- U3 pad 33: (no net) -> /SOLAR_1
- U3 pad 42: /RFM_RESET -> Net-(J7-Pad1)
- U3 pad 9: (no net) -> Net-(J9-Pad1)
